File: pcbs/numpad-wired.kicad_pcb (KiCad board)
At the start: 2 copper layers, 77.7 x 77.7 mm, 15 parts

Commit message: added mounting holes, and reset switch to both
Parts:
- added H2: , smd2:mounting_hole_plated, F.Cu at (97.7, 121.8)
- added H2: , smd2:mounting_hole_plated, F.Cu at (158.9, 124.9)
- added H2: , smd2:mounting_hole_plated, F.Cu at (158.6, 57.3)
- added H2: , smd2:mounting_hole_plated, F.Cu at (126.4, 57.2)
- added RST1: , smd2:reset_switch_smd_side, F.Cu at (114.8, 54.4)
Routing:
- net RST: track 0.00 -> 12.2 mm
