File: pcbs/numpad-wireless.kicad_pcb (KiCad board)
At the start: 2 copper layers, 77.7 x 77.7 mm, 17 parts

Commit message: added mounting holes + reformatted
Parts:
- added H2: , smd2:mounting_hole_plated, F.Cu at (157.4, 57.7)
- added H2: , smd2:mounting_hole_plated, F.Cu at (158.4, 124.4)
- added H2: , smd2:mounting_hole_plated, F.Cu at (106.2, 74.0)
- added H2: , smd2:mounting_hole_plated, F.Cu at (97.4, 123.8)

Commit message: added mounting holes, and reset switch to both
Parts:
- moved H2 24.5 mm to (127.2, 61.3)
Changed lines of the file:
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@@
 	(footprint "smd2:mounting_hole_plated"
 		(layer "F.Cu")
-		(at 106.24 73.97)
+		(at 127.24 61.34)
 		(property "Reference" "H2"
 			(at 0 3 0)
